File: Eagle_Files/FemtoBeacon_r2.0.0/femtoBeacon_r2.0.1.brd (EAGLE design)
At the start: 18 x 18 mm, 60 parts

Commit message: Revision 2.0.7 of the coin, with USB Host and RGB LED, plus u.FL connector
Parts:
- renumbered U$12 to BAL, U$44 to BARO, U$6 to IMU, U$76 to IC
