File: Eagle_Files/FemtoBeacon_r2.0.0/femtoBeacon_dongle_r2.0.6_RGB.sch (EAGLE design)
At the start: 73 parts

Commit message: Adding FemtoBeacon coin r2.0.7, and FemtoBeacon dongle r2.0.6
Parts:
- removed ANT_SMD: 0479480001, molex-antenna-2.4GHz:0479480001
- removed BALUN: JOHANSON_2450BM15A0015E, balun:JOHANSON_2450BM15A0015E
- removed BARO: MS5611-01BA03, freeimu:MS5611-01BA03
- removed C12: 22pF, parts_0201:CAPACITOR_0201
- removed C29, C30, C32: 0.1uF, parts_0201:CAPACITOR_0201
- removed C31: 10nF, parts_0201:CAPACITOR_0201
- removed FID4, FID5, FID6: FIDUCIAL, adafruit:FIDUCIAL
- removed IMU: MPU-9250, mpu9250:MPU-9250
- removed R10: 100K, parts_0201:RESISTOR_0201
- removed R3: 330, microbuilder:RESISTOR_0402
- removed R5: 330, parts_0201:RESISTOR_0201
- removed R8, R9: 2.2K, parts_0201:RESISTOR_0201
- removed U$10, U$2, U$35, U$36, U$37, U$38, U$39, U$43, U$45, U$46, U$47, U$48, U$5, U$54, U$7, U$9: 1X1_ROUND, pins_1.27mm_pitch:1X1_ROUND
- removed USB: USB_MICROB, femtoduino:USB_MICROB
- added C24: 22pF, parts_0201:CAPACITOR_0201
- added CN1: (no value), microbuilder:USB_TYPEA
- added FB2: (no value), microbuilder:FERRITE_0603MP
- added U$12: JOHANSON_2450BM15A0015E, balun:JOHANSON_2450BM15A0015E
- added U$6: 0479480001, molex-antenna-2.4GHz:0479480001
- ASWITCH: MFR_ID (none) -> AS222-92LF
- C1, C10, C16, C17, C8, C9: DIGIKEY_PART 490-3194-1-ND -> (none); MFR_ID (none) -> GRM033C80J104KE84D
- C11: MFR_ID (none) -> GRM1555C1H1R2BA01D
- C13: DIGIKEY_PART 490-3194-1-ND -> (none)
- C14, C15: MFR_ID (none) -> C0603C0G1E090B030BG
- C18, C19, C20, C23: DIGIKEY_PART 490-3194-1-ND -> (none); MFR_ID (none) -> GRM0335C1E220JA01D
- C2: MFR_ID (none) -> GRM033C80J104KE84D
- C21, C22: MFR_ID (none) -> AMK105CBJ106MV-F
- C5, C6: MFR_ID (none) -> C1005X5R1A225K050BC
- C7: MFR_ID (none) -> C0603X5R0J474K030BC
- FB1: value Ferrite -> (none); MFR_ID (none) -> BLM18RK102SN1D
- L6: MFR_ID (none) -> LQM18FN100M00D
- LDO_VREG: MFR_ID (none) -> MCP1700T-3302E/TT
- R1, R4, R6, R7: MFR_ID (none) -> CRCW0201330RJNED
- R2: MFR_ID (none) -> RC0402FR-0710KL
- U$1: value 1X1_ROUND -> 1X5_ROUND; device pins_1.27mm_pitch:1X1_ROUND -> pins_fine_pitch:1X5_ROUND
- U$76: MFR_ID (none) -> ATSAMR21E18A-MFT
- UFLANT: MFR_ID (none) -> 734120110
- XOSCRF: MFR_ID (none) -> TSX-3225 16.0000MF09Z-AC0
- renumbered IC to U$76
Connections:
- removed net N$1: R10.1, R5.2, USB.ID
- removed net PA18/FSYNC: IMU.FSYNC, R3.2, U$36.1, U$76.PA18
- removed net PA19/INTA: IMU.INT, U$35.1, U$76.PA19
- new net PA18/INTA: U$76.PA18
- new net PA19/FSYNC: U$76.PA19
- net 3.3V: now also U$1.2; no longer BARO.PS, BARO.VDD, C29.P$1, C30.P$2, C31.P$2, IMU.NCS, IMU.RESV@1, IMU.VDD, IMU.VDDIO, R10.2, R8.2, R9.2, U$5.1
- net ANT_LINE: now also L1.1, U$6.1; no longer ANT_SMD.1, L1.2
- net ANT_OUT: now also C18.P$1, U$12.1; no longer BALUN.1, C12.P$1
- net ANT_SMD: now also C24.P$2, L1.2; no longer C23.P$2, L1.1
- net ANT_UFL: now also C23.P$1; no longer C20.P$1
- net GND: now also C19.P$1, C20.P$2, U$1.1, U$12.2, U$12.5, U$12.6; no longer BALUN.2, BALUN.5, BALUN.6, BARO.CSB, BARO.CSB1, BARO.GND, C18.P$1, C19.P$2, C29.P$2, C30.P$1, C31.P$1, C32.P$2, IMU.RESV@20, R3.1, U$2.1
- net N$4: now also CN1.VBUS, FB2.P$1; no longer C32.P$1, IMU.REGOUT
- net N$5: now also CN1.GND; no longer USB.GND@1, USB.GND@2, USB.GND@3, USB.GND@4, USB.GND@5, USB.GND@6, USB.GND@7
- net PA06(R): no longer U$54.1
- net PA07(G): no longer U$43.1
- net PA08/I2C/SDA: now also C20.P$1; no longer C19.P$1
- net PA09/I2C/SCL: now also C19.P$2; no longer C18.P$2
- net PA15/XOUT_MC/TX: no longer U$39.1
- net PA16/I2C: no longer BARO.SDI/SDA, IMU.SDA/SDI, R8.1, U$38.1
- net PA17/I2C: no longer BARO.SCLK, IMU.SCL/SCLK, R9.1, U$37.1
- net PA24/USBDM: now also CN1.D-; no longer U$9.1, USB.D-
- net PA25/USBDP: now also CN1.D+; no longer U$10.1, USB.D+
- net PA27(B): no longer U$7.1
- net PA28: no longer R5.1, U$48.1
- net PA30/SWCLK: now also U$1.4; no longer U$46.1
- net PA31/SWDIO: now also U$1.5; no longer U$47.1
- net RESET: now also U$1.3; no longer U$45.1
- net RFN: now also U$12.3; no longer BALUN.3
- net RFP: now also U$12.4; no longer BALUN.4
- net RFSWITCH_PIN1: now also C24.P$1; no longer C23.P$1
- net RFSWITCH_PIN3: now also C23.P$2; no longer C20.P$2
- net RFSWITCH_PIN5: now also C18.P$2; no longer C12.P$2
- net VIN: now also FB2.P$2; no longer U$1.1, USB.V
Other:
- note removed: "2.0.2 - Pin names FSYNC and IN on PA18 were swapped. Needed correction in schematic only. PA18 is FSYNC, PA19 is INT"
- note removed: "FSYNC"
- note removed: "INTA"
- note removed: "SCL"
- note removed: "SDA"
