File: Eagle_Files/FemtoBeacon_ESP32_Coin_r1.0.0/femto-beacon-esp32coin.sch (EAGLE design)
At the start: 48 parts, among them IC1 ESP32-QFN_5X5

Commit message: Fixing solder stop mask on femto-beacon-esp32coin and femto-beacon-esp32-lps. Adding Blender3D model of stencil jig for the coin
Connections:
- net 3.3V: now also RGB1.GND
- net GND: no longer RGB1.GND
Changed lines of the file:
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@@
 <attribute name="MPN" value="RC0201FR-07270RL"/>
 </part>
-<part name="U$25" library="microbuilder" deviceset="GND" device=""/>
 <part name="U$35" library="microbuilder" deviceset="GND" device=""/>
 <part name="U$36" library="microbuilder" deviceset="3.3V" device=""/>
@@
 <part name="U$3" library="microbuilder" deviceset="GND" device=""/>
 <part name="R6" library="parts_0201" deviceset="RESISTOR_0201" device="" value="DNP"/>
+<part name="U$9" library="microbuilder" deviceset="3.3V" device=""/>
 </parts>
 <sheets>
@@
 <attribute name="MPN" x="198.12" y="144.78" size="1.778" layer="96" rot="R180" display="off"/>
 </instance>
-<instance part="U$25" gate="G$1" x="210.82" y="149.86" smashed="yes" rot="R180">
-<attribute name="VALUE" x="212.344" y="152.4" size="1.27" layer="96" rot="R180"/>
-</instance>
 <instance part="U$35" gate="G$1" x="203.2" y="73.66" smashed="yes" rot="R270">
 <attribute name="VALUE" x="200.66" y="75.184" size="1.27" layer="96" rot="R270"/>
@@
 <attribute name="NAME" x="43.815" y="119.38" size="1.016" layer="95" font="vector" rot="R90"/>
 <attribute name="VALUE" x="48.895" y="119.38" size="1.016" layer="96" font="vector" rot="R90"/>
+</instance>
+<instance part="U$9" gate="G$1" x="213.36" y="149.86" smashed="yes">
+<attribute name="VALUE" x="211.836" y="150.876" size="1.27" layer="96"/>
 </instance>
 </instances>
@@
 <pinref part="U$34" gate="G$1" pin="GND"/>
 <wire x1="27.94" y1="45.72" x2="27.94" y2="43.18" width="0.1524" layer="91"/>
-</segment>
-<segment>
-<pinref part="RGB1" gate="G$1" pin="GND"/>
-<wire x1="213.36" y1="147.32" x2="210.82" y2="147.32" width="0.1524" layer="91"/>
-<pinref part="U$25" gate="G$1" pin="GND"/>
 </segment>
 <segment>
@@
 <wire x1="200.66" y1="76.2" x2="220.98" y2="76.2" width="0.1524" layer="91"/>
 </segment>
-</net>
+<segment>
+<pinref part="RGB1" gate="G$1" pin="GND"/>
+<pinref part="U$9" gate="G$1" pin="3.3V"/>
+</segment>
+</net>

Commit message: Setting correct ESP32 chip for the coin design to ESP32‑D2WD as it has 2MiB of internal Flash
Parts:
- IC1: MPN (none) -> ESP32-D2WD
Connections:
- net EN renamed RESET
Changed lines of the file:
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@@
 <part name="FRAME2" library="frames" library_urn="urn:adsk.eagle:library:229" deviceset="LETTER_L" device=""/>
 <part name="FRAME3" library="frames" library_urn="urn:adsk.eagle:library:229" deviceset="LETTER_L" device=""/>
-<part name="IC1" library="esp32-wroom-32" deviceset="ESP32-QFN_5X5" device=""/>
+<part name="IC1" library="esp32-wroom-32" deviceset="ESP32-QFN_5X5" device="">
+<attribute name="MPN" value="ESP32-D2WD"/>
+</part>
 <part name="U$1" library="microbuilder" deviceset="3.3V" device=""/>
 <part name="U$2" library="microbuilder" deviceset="VIN" device=""/>
@@
 <attribute name="DRAWING_NAME" x="165.1" y="19.05" size="2.54" layer="94"/>
 </instance>
-<instance part="IC1" gate="G$1" x="127" y="111.76" smashed="yes"/>
+<instance part="IC1" gate="G$1" x="127" y="111.76" smashed="yes">
+<attribute name="MPN" x="127" y="111.76" size="1.778" layer="96" display="off"/>
+</instance>
 <instance part="U$1" gate="G$1" x="185.42" y="129.54" smashed="yes" rot="R270">
 <attribute name="VALUE" x="186.436" y="131.064" size="1.27" layer="96" rot="R270"/>
@@
 </segment>
 </net>
-<net name="EN" class="0">
+<net name="RESET" class="0">
 <segment>
 <pinref part="IC1" gate="G$1" pin="CHIP_PU"/>
