File: Eagle_Files/FemtoBeacon_ESP32_Coin_r1.0.0/femto-beacon-esp32coin.sch (EAGLE design)
At the start: 48 parts, among them IC1 ESP32-QFN_5X5

Commit message: Current work on Hacker House board, and ESP32 coins
Parts:
- FB1, FB2: value (none) -> FERRITE
Changed lines of the file:
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@@
 </part>
 <part name="U$16" library="microbuilder" deviceset="GND" device=""/>
-<part name="FB1" library="microbuilder" deviceset="FERRITE" device="_0603MP"/>
-<part name="FB2" library="microbuilder" deviceset="FERRITE" device="_0603MP"/>
+<part name="FB1" library="microbuilder" deviceset="FERRITE" device="_0603MP" value="FERRITE"/>
+<part name="FB2" library="microbuilder" deviceset="FERRITE" device="_0603MP" value="FERRITE"/>
 <part name="U$6" library="microbuilder" deviceset="3.3V" device=""/>
 <part name="U$17" library="microbuilder" deviceset="GND" device=""/>
