File: Eagle_Files/FemtoBeacon_ESP32_Coin_r1.0.0/femto-beacon-esp32pico-d4-coin-imu.brd (EAGLE design)
At the start: 26.2 x 29.2 mm, 36 parts, among them IC1 ESP32-PICO-D4

Commit message: Current work on Hacker House board, and ESP32 coins
Parts:
- added ALT1: MS5611-01BA03, freeimu:MS5611-01BA03
- added C1, C6: 1uF, parts_0201:PART
- added C25, C28, C29: 0.1uF, parts_0201:PART
- added IMU1: ICM-20948, icm-20948:QFN24_3X3
- added LDO1.8V: NCP705MT18TCG, onsemi:CASE_511BR
- added LVL_SHFT: SN74AVC4T774RSVR, til-level-shifter:RSV16
- added R1: 10K, parts_0201:PART
- added U$1: 1X2_ROUND, pins_1.27mm_pitch:1X2_ROUND
Connections:
- removed net IO23: IC1.36
- removed net IO25: IC1.14
- removed net IO27: IC1.16
- new net 1.8V: C1.2, C28.2, IMU1.13, IMU1.8, LDO1.8V.1, LVL_SHFT.13
- new net B_MTCK/HSPID(MOSI): IMU1.24, LVL_SHFT.9
- new net B_MTDI/HSPIQ(MISO): IMU1.9, LVL_SHFT.12
- new net B_MTDO/HSPICS0(CS): IMU1.22, LVL_SHFT.11
- new net B_MTMS/HSPI_CLK: IMU1.23, LVL_SHFT.10
- new net INT_WAKE_IMU: IMU1.12, U$1.P$1
- new net IO25/OE_1.8V: IC1.14, LVL_SHFT.7, R1.1
- new net IO27/CS_ALTI: ALT1.4, IC1.16
- new net N$16: C29.2, IMU1.10
- new net ON_1.8V: IC1.36, LDO1.8V.4
- net 3.3V: now also ALT1.1, C25.1, C6.2, LDO1.8V.6, LVL_SHFT.14, LVL_SHFT.16, LVL_SHFT.5, LVL_SHFT.6, R1.2
- net GND: now also ALT1.2, ALT1.3, C1.1, C25.2, C28.1, C29.1, C6.1, IMU1.11, IMU1.18, IMU1.20, LDO1.8V.3, LVL_SHFT.15, LVL_SHFT.8
- net MTCK/HSPID(MOSI): now also ALT1.7, LVL_SHFT.4
- net MTDI/HSPIQ(MISO): now also ALT1.6, LVL_SHFT.1
- net MTDO/HSPICS0(CS): now also LVL_SHFT.2
- net MTMS/HSPI_CLK: now also ALT1.8, LVL_SHFT.3
Routing:
- net MTDI/HSPIQ(MISO): track 5.11 -> 42.2 mm, vias 0 -> 2
- net GND: track 76.4 -> 106.9 mm
- net 3.3V: track 48.7 -> 78.7 mm, vias 6 -> 9
- net 1.8V: track 0.00 -> 27.1 mm, vias 0 -> 3
- net B_MTDI/HSPIQ(MISO): track 0.00 -> 16.7 mm, vias 0 -> 2
- net IO25/OE_1.8V: track 0.00 -> 15.2 mm, vias 0 -> 2
- net MTCK/HSPID(MOSI): track 10.9 -> 24.0 mm
- net MTMS/HSPI_CLK: track 5.94 -> 19.0 mm
- net IO27/CS_ALTI: track 0.00 -> 11.5 mm, vias 0 -> 1
- net INT_WAKE_IMU: track 0.00 -> 9.70 mm, vias 0 -> 1
- net MTDO/HSPICS0(CS): track 8.37 -> 17.8 mm
- net ON_1.8V: track 0.00 -> 5.31 mm, vias 0 -> 1
- net B_MTDO/HSPICS0(CS): track 0.00 -> 3.60 mm
- net B_MTMS/HSPI_CLK: track 0.00 -> 3.07 mm
- net N$16: track 0.00 -> 1.97 mm
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