File: Eagle_Files/FemtoBeacon_ESP32_Coin_r1.0.0/femto-beacon-esp32pico-d4-coin-imu.sch (EAGLE design)
At the start: 50 parts, among them IC1 ESP32-PICO-D4

Commit message: Current work on Hacker House board, and ESP32 coins
Parts:
- removed LPS1: DWM100, decawave:DWM100
- removed R7: 4.7K, parts_0201:RESISTOR_0201
- removed U$39: 1X4_ROUND, pins_1.27mm_pitch:1X4_ROUND
Connections:
- removed net EXTON_DECA: LPS1.EXTON, U$39.1
- removed net IO18/CS_DECA: IC1.IO18/VSPICLK, LPS1.SPICS
- removed net IRQ_DECA: LPS1.IRQ/GPIO8, R7.1, U$39.4
- removed net RST_DECA: LPS1.RST, U$39.3
- removed net WAKE_DECA: LPS1.WAKEUP, U$39.2
- new net IO18: IC1.IO18/VSPICLK
- net 3.3V: no longer LPS1.3V3@1, LPS1.3V3@2, LPS1.VDDAON
- net GND: no longer LPS1.VSS@1, LPS1.VSS@2, LPS1.VSS@3, LPS1.VSS@4, LPS1.VSS@5, R7.2
- net MTCK/HSPID(MOSI): no longer LPS1.SPIMOSI
- net MTDI/HSPIQ(MISO): no longer LPS1.SPIMISO
- net MTMS/HSPI_CLK: no longer LPS1.SPICLK
Other:
- note removed: "UWB - LPS"
Changed lines of the file:
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@@
 <part name="FID4" library="adafruit" deviceset="FIDUCIAL" device=""/>
 <part name="FID5" library="adafruit" deviceset="FIDUCIAL" device=""/>
-<part name="FRAME3" library="frames" library_urn="urn:adsk.eagle:library:229" deviceset="LETTER_L" device=""/>
-<part name="LPS1" library="decawave" deviceset="DWM100" device=""/>
-<part name="U$11" library="microbuilder" deviceset="3.3V" device=""/>
-<part name="U$23" library="microbuilder" deviceset="GND" device=""/>
-<part name="U$24" library="microbuilder" deviceset="GND" device=""/>
-<part name="U$37" library="microbuilder" deviceset="GND" device=""/>
-<part name="R7" library="parts_0201" deviceset="RESISTOR_0201" device="" value="4.7K">
-<attribute name="MPN" value="RC0201FR-074K7L"/>
-</part>
-<part name="U$38" library="microbuilder" deviceset="GND" device=""/>
-<part name="U$39" library="pins_1.27mm_pitch" deviceset="1X4_ROUND" device=""/>
 <part name="FID6" library="adafruit" deviceset="FIDUCIAL" device=""/>
 <part name="U$7" library="microbuilder" deviceset="1.8V" device=""/>
@@
 </segment>
 </bus>
-<bus name="IO18/CS_DECA,IO27/CS_ALTI">
+<bus name="IO18,IO27/CS_ALTI">
 <segment>
 <wire x1="78.74" y1="66.04" x2="93.98" y2="66.04" width="0.762" layer="92"/>
@@
 </segment>
 </net>
-<net name="IO18/CS_DECA" class="0">
+<net name="IO18" class="0">
 <segment>
 <pinref part="IC1" gate="G$1" pin="IO18/VSPICLK"/>
@@
 </segment>
 </bus>
-<bus name="IO18/CS_DECA,IO27/CS_ALTI">
+<bus name="IO18,IO27/CS_ALTI">
 <segment>
 <wire x1="210.82" y1="129.54" x2="210.82" y2="114.3" width="0.762" layer="92"/>
@@
 </segment>
 </net>
-<net name="IO18/CS_DECA" class="0">
+<net name="IO18" class="0">
 <segment>
 <wire x1="210.82" y1="124.46" x2="223.52" y2="124.46" width="0.1524" layer="91"/>
@@
 </segment>
 </net>
-</nets>
-</sheet>
-<sheet>
-<plain>
-<text x="5.08" y="170.18" size="7.62" layer="94">UWB - LPS</text>
-</plain>
-<instances>
-<instance part="FRAME3" gate="G$1" x="0" y="0" smashed="yes"/>
-<instance part="LPS1" gate="G$1" x="76.2" y="109.22" smashed="yes"/>
-<instance part="U$11" gate="G$1" x="38.1" y="104.14" smashed="yes" rot="R90">
-<attribute name="VALUE" x="37.084" y="102.616" size="1.27" layer="96" rot="R90"/>
-</instance>
-<instance part="U$23" gate="G$1" x="35.56" y="99.06" smashed="yes" rot="R270">
-<attribute name="VALUE" x="33.02" y="100.584" size="1.27" layer="96" rot="R270"/>
-</instance>
-<instance part="U$24" gate="G$1" x="86.36" y="76.2" smashed="yes">
-<attribute name="VALUE" x="84.836" y="73.66" size="1.27" layer="96"/>
-</instance>
-<instance part="U$37" gate="G$1" x="106.68" y="119.38" smashed="yes" rot="R90">
-<attribute name="VALUE" x="109.22" y="117.856" size="1.27" layer="96" rot="R90"/>
-</instance>
-<instance part="R7" gate="G$1" x="124.46" y="111.76" smashed="yes">
-<attribute name="NAME" x="124.46" y="113.665" size="1.016" layer="95" font="vector"/>
-<attribute name="VALUE" x="124.46" y="108.585" size="1.016" layer="96" font="vector"/>
-<attribute name="MPN" x="124.46" y="111.76" size="1.778" layer="96" display="off"/>
-</instance>
-<instance part="U$38" gate="G$1" x="134.62" y="111.76" smashed="yes" rot="R90">
-<attribute name="VALUE" x="137.16" y="110.236" size="1.27" layer="96" rot="R90"/>
-</instance>
-<instance part="U$39" gate="G$1" x="185.42" y="134.62" smashed="yes"/>
-</instances>
-<busses>
-<bus name="SPI:MTCK/HSPID(MOSI),MTDI/HSPIQ(MISO),MTDO/HSPICS0(CS),MTMS/HSPI_CLK">
-<segment>
-<wire x1="170.18" y1="111.76" x2="185.42" y2="111.76" width="0.762" layer="92"/>
-<label x="190.5" y="111.76" size="1.778" layer="95"/>
-</segment>
-</bus>
-<bus name="IO18/CS_DECA,IO27/CS_ALTI">
-<segment>
-<wire x1="137.16" y1="55.88" x2="152.4" y2="55.88" width="0.762" layer="92"/>
-<label x="134.62" y="60.96" size="1.778" layer="95" rot="R180"/>
-</segment>
-</bus>
-</busses>
-<nets>
-<net name="MTMS/HSPI_CLK" class="0">
-<segment>
-<wire x1="170.18" y1="111.76" x2="170.18" y2="106.68" width="0.1524" layer="91"/>
-<label x="170.18" y="83.82" size="1.778" layer="95" rot="R270"/>
-<pinref part="LPS1" gate="G$1" pin="SPICLK"/>
-<wire x1="170.18" y1="106.68" x2="170.18" y2="86.36" width="0.1524" layer="91"/>
-<wire x1="93.98" y1="106.68" x2="170.18" y2="106.68" width="0.1524" layer="91"/>
-<junction x="170.18" y="106.68"/>
-</segment>
-</net>
-<net name="MTDI/HSPIQ(MISO)" class="0">
-<segment>
-<wire x1="172.72" y1="111.76" x2="172.72" y2="104.14" width="0.1524" layer="91"/>
-<label x="172.72" y="83.82" size="1.778" layer="95" rot="R270"/>
-<pinref part="LPS1" gate="G$1" pin="SPIMISO"/>
-<wire x1="172.72" y1="104.14" x2="172.72" y2="86.36" width="0.1524" layer="91"/>
-<wire x1="93.98" y1="104.14" x2="172.72" y2="104.14" width="0.1524" layer="91"/>
-<junction x="172.72" y="104.14"/>
-</segment>
-</net>
-<net name="MTCK/HSPID(MOSI)" class="0">
-<segment>
-<wire x1="175.26" y1="111.76" x2="175.26" y2="101.6" width="0.1524" layer="91"/>
-<label x="175.26" y="83.82" size="1.778" layer="95" rot="R270"/>
-<pinref part="LPS1" gate="G$1" pin="SPIMOSI"/>
-<wire x1="175.26" y1="101.6" x2="175.26" y2="86.36" width="0.1524" layer="91"/>
-<wire x1="93.98" y1="101.6" x2="175.26" y2="101.6" width="0.1524" layer="91"/>
-<junction x="175.26" y="101.6"/>
-</segment>
-</net>
-<net name="EXTON_DECA" class="0">
-<segment>
-<pinref part="LPS1" gate="G$1" pin="EXTON"/>
-<wire x1="58.42" y1="119.38" x2="48.26" y2="119.38" width="0.1524" layer="91"/>
-<label x="45.72" y="119.38" size="1.778" layer="95" rot="R180"/>
-</segment>
-<segment>
-<pinref part="U$39" gate="G$1" pin="1"/>
-<wire x1="185.42" y1="134.62" x2="180.34" y2="134.62" width="0.1524" layer="91"/>
-<label x="177.8" y="134.62" size="1.778" layer="95" rot="R180"/>
-</segment>
-</net>
-<net name="WAKE_DECA" class="0">
-<segment>
-<pinref part="LPS1" gate="G$1" pin="WAKEUP"/>
-<wire x1="58.42" y1="116.84" x2="48.26" y2="116.84" width="0.1524" layer="91"/>
-<label x="45.72" y="116.84" size="1.778" layer="95" rot="R180"/>
-</segment>
-<segment>
-<pinref part="U$39" gate="G$1" pin="2"/>
-<wire x1="185.42" y1="132.08" x2="180.34" y2="132.08" width="0.1524" layer="91"/>
-<label x="177.8" y="132.08" size="1.778" layer="95" rot="R180"/>
-</segment>
-</net>
-<net name="RST_DECA" class="0">
-<segment>
-<pinref part="LPS1" gate="G$1" pin="RST"/>
-<wire x1="58.42" y1="114.3" x2="48.26" y2="114.3" width="0.1524" layer="91"/>
-<label x="45.72" y="114.3" size="1.778" layer="95" rot="R180"/>
-</segment>
-<segment>
-<pinref part="U$39" gate="G$1" pin="3"/>
-<wire x1="185.42" y1="129.54" x2="180.34" y2="129.54" width="0.1524" layer="91"/>
-<label x="177.8" y="129.54" size="1.778" layer="95" rot="R180"/>
-</segment>
-</net>
-<net name="GND" class="0">
-<segment>
-<pinref part="LPS1" gate="G$1" pin="VSS@1"/>
-<pinref part="U$23" gate="G$1" pin="GND"/>
-<wire x1="38.1" y1="99.06" x2="58.42" y2="99.06" width="0.1524" layer="91"/>
-</segment>
-<segment>
-<pinref part="LPS1" gate="G$1" pin="VSS@2"/>
-<pinref part="U$24" gate="G$1" pin="GND"/>
-<wire x1="86.36" y1="78.74" x2="86.36" y2="83.82" width="0.1524" layer="91"/>
-</segment>
-<segment>
-<pinref part="LPS1" gate="G$1" pin="VSS@3"/>
-<wire x1="93.98" y1="111.76" x2="99.06" y2="111.76" width="0.1524" layer="91"/>
-<wire x1="99.06" y1="111.76" x2="99.06" y2="116.84" width="0.1524" layer="91"/>
-<pinref part="LPS1" gate="G$1" pin="VSS@4"/>
-<wire x1="99.06" y1="116.84" x2="93.98" y2="116.84" width="0.1524" layer="91"/>
-<pinref part="LPS1" gate="G$1" pin="VSS@5"/>
-<wire x1="93.98" y1="119.38" x2="99.06" y2="119.38" width="0.1524" layer="91"/>
-<wire x1="99.06" y1="119.38" x2="99.06" y2="116.84" width="0.1524" layer="91"/>
-<junction x="99.06" y="116.84"/>
-<wire x1="99.06" y1="119.38" x2="104.14" y2="119.38" width="0.1524" layer="91"/>
-<junction x="99.06" y="119.38"/>
-<pinref part="U$37" gate="G$1" pin="GND"/>
-</segment>
-<segment>
-<pinref part="R7" gate="G$1" pin="2"/>
-<pinref part="U$38" gate="G$1" pin="GND"/>
-</segment>
-</net>
-<net name="3.3V" class="0">
-<segment>
-<pinref part="LPS1" gate="G$1" pin="3V3@2"/>
-<pinref part="LPS1" gate="G$1" pin="3V3@1"/>
-<wire x1="58.42" y1="101.6" x2="58.42" y2="104.14" width="0.1524" layer="91"/>
-<pinref part="LPS1" gate="G$1" pin="VDDAON"/>
-<wire x1="58.42" y1="104.14" x2="58.42" y2="106.68" width="0.1524" layer="91"/>
-<junction x="58.42" y="104.14"/>
-<pinref part="U$11" gate="G$1" pin="3.3V"/>
-<wire x1="58.42" y1="104.14" x2="40.64" y2="104.14" width="0.1524" layer="91"/>
-</segment>
-</net>
-<net name="IRQ_DECA" class="0">
-<segment>
-<pinref part="LPS1" gate="G$1" pin="IRQ/GPIO8"/>
-<wire x1="93.98" y1="114.3" x2="121.92" y2="114.3" width="0.1524" layer="91"/>
-<pinref part="R7" gate="G$1" pin="1"/>
-<wire x1="121.92" y1="114.3" x2="142.24" y2="114.3" width="0.1524" layer="91"/>
-<wire x1="121.92" y1="111.76" x2="121.92" y2="114.3" width="0.1524" layer="91"/>
-<junction x="121.92" y="114.3"/>
-<label x="144.78" y="114.3" size="1.778" layer="95"/>
-</segment>
-<segment>
-<pinref part="U$39" gate="G$1" pin="4"/>
-<wire x1="185.42" y1="127" x2="180.34" y2="127" width="0.1524" layer="91"/>
-<label x="177.8" y="127" size="1.778" layer="95" rot="R180"/>
-</segment>
-</net>
-<net name="IO27/CS_ALTI" class="0">
-<segment>
-<label x="139.7" y="68.58" size="1.778" layer="95" rot="R90"/>
-<wire x1="139.7" y1="66.04" x2="139.7" y2="55.88" width="0.1524" layer="91"/>
-</segment>
-</net>
-<net name="IO18/CS_DECA" class="0">
-<segment>
-<label x="142.24" y="68.58" size="1.778" layer="95" rot="R90"/>
-<wire x1="142.24" y1="66.04" x2="142.24" y2="60.96" width="0.1524" layer="91"/>
-<pinref part="LPS1" gate="G$1" pin="SPICS"/>
-<wire x1="142.24" y1="60.96" x2="142.24" y2="55.88" width="0.1524" layer="91"/>
-<wire x1="93.98" y1="99.06" x2="149.86" y2="99.06" width="0.1524" layer="91"/>
-<wire x1="149.86" y1="99.06" x2="149.86" y2="60.96" width="0.1524" layer="91"/>
-<wire x1="149.86" y1="60.96" x2="142.24" y2="60.96" width="0.1524" layer="91"/>
-<junction x="142.24" y="60.96"/>
-</segment>
-</net>
