File: Eagle_Files/FemtoBeacon_ESP32_Coin_r1.0.0/femto-beacon-esp32pico-d4-lps.brd (EAGLE design)
At the start: 38.9 x 29.2 mm, 46 parts, among them IC1 ESP32-PICO-D4

Commit message: Current work on Hacker House board, and ESP32 coins
Parts:
- removed SJ_FSYNC: DNP, microbuilder:SOLDERJUMPER_CLOSEDWIRE
- added C1, C6: 1uF, parts_0201:PART
- added LDO1.8V: NCP705MT18TCG, onsemi:CASE_511BR
- added LVL_SHFT: SN74AVC4T774RSVR, til-level-shifter:RSV16
- added R1: 10K, parts_0201:PART
- moved C4 0.36 mm to (7.87, 16.3), turned to 0 degrees
- moved C8 0.18 mm to (10.4, 7.37)
- moved C25 0.16 mm to (15.0, 13.7)
- moved ALT1 0.13 mm to (13.0, 12.6)
- moved L2 0.13 mm to (9.40, 7.37)
Connections:
- removed net FSYNC_IMU: IMU1.11, SJ_FSYNC.1, U$1.P$2
- removed net IO25: IC1.14
- new net 1.8V: C1.2, C28.2, IMU1.13, IMU1.8, LDO1.8V.1, LVL_SHFT.13
- new net B_MTCK/HSPID(MOSI): IMU1.24, LVL_SHFT.9
- new net B_MTDI/HSPIQ(MISO): IMU1.9, LVL_SHFT.12
- new net B_MTDO/HSPICS0(CS): IMU1.22, LVL_SHFT.11
- new net B_MTMS/HSPI_CLK: IMU1.23, LVL_SHFT.10
- new net IO25/OE_1.8V: IC1.14, LVL_SHFT.7, R1.1
- new net ON_1.8V: IC1.36, LDO1.8V.4
- net 3.3V: now also C6.2, LDO1.8V.6, LVL_SHFT.14, LVL_SHFT.16, LVL_SHFT.5, LVL_SHFT.6, R1.2; no longer C28.2, IMU1.13, IMU1.8
- net GND: now also C1.1, C6.1, IMU1.11, LDO1.8V.3, LVL_SHFT.15, LVL_SHFT.8; no longer SJ_FSYNC.2
- net MTCK/HSPID(MOSI): now also LVL_SHFT.4; no longer IMU1.24
- net MTDI/HSPIQ(MISO): now also LVL_SHFT.1; no longer IMU1.9
- net MTDO/HSPICS0(CS): now also LVL_SHFT.2; no longer IMU1.22
- net MTMS/HSPI_CLK: now also LVL_SHFT.3; no longer IMU1.23
Routing:
- net GND: track 123.1 -> 155.2 mm, vias 12 -> 11
- net 1.8V: track 0.00 -> 27.1 mm, vias 0 -> 3
- net FSYNC_IMU: track 21.9 -> 0.00 mm, vias 2 -> 0
- net B_MTDI/HSPIQ(MISO): track 0.00 -> 16.7 mm, vias 0 -> 2
- net IO25/OE_1.8V: track 0.00 -> 15.2 mm, vias 0 -> 2
- net 3.3V: track 86.1 -> 99.2 mm, vias 9 -> 10
- net MTDI/HSPIQ(MISO): track 44.6 -> 55.9 mm, vias 2 -> 3
- net MTDO/HSPICS0(CS): track 24.2 -> 17.8 mm
- net MTMS/HSPI_CLK: track 37.3 -> 31.8 mm
- net ON_1.8V: track 0.00 -> 5.31 mm, vias 0 -> 1
- net MTCK/HSPID(MOSI): track 43.8 -> 38.6 mm
- net B_MTDO/HSPICS0(CS): track 0.00 -> 3.60 mm
- net B_MTMS/HSPI_CLK: track 0.00 -> 3.07 mm
- net B_MTCK/HSPID(MOSI): track 0.00 -> 1.93 mm
- net IO0/BOOT: track 19.5 -> 18.5 mm
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Other:
- board text added: "2.0.1"
- board text removed: "2.0.0"
